Commit message: add localization

File: turtlebot_description/urdf/turtlebot3_burger.urdf.xacro (robot description, xacro)
@@ -9,4 +9,10 @@
     <origin xyz="0.0 0.0 0.010" rpy="0 0 0"/>
   </joint>
+<!--
+  <joint name="base_joint" type="fixed">
+    <parent link="base_link"/>
+    <child link="base_footprint"/>
+    <origin xyz="0.0 0.0 -0.010" rpy="0 0 0"/>
+  </joint> -->
   <link name="base_link">
     <visual>
@@ -113,5 +119,5 @@
   </joint>
   <link name="imu_link"/>
-  <joint name="scan_joint" type="fixed">
+  <!-- <joint name="scan_joint" type="fixed">
     <parent link="base_link"/>
     <child link="base_scan"/>
@@ -139,4 +145,4 @@
                izz="0.001" />
     </inertial>
-  </link>
+  </link> -->
 </robot>
